File: stm8s-core-board.sch (KiCad schematic (older format))
At the start: 21 parts, among them IC1 STM8S003F3P, P1 CONN_01X06, P2 USB_OTG, P3 CONN_01X09, P4 CONN_01X09, P5 CONN_01X02, SW1 SW_PUSH, U1 AS1117-5.0, Y1 16MHz

Commit message: forgot commit for long time. don't know what changed
Parts:
- removed C4, C5: 22pF, Capacitors_SMD:C_0603_HandSoldering, symbol C_Small
- removed IC1: STM8S003F3P, Housings_SSOP:TSSOP-20_4.4x6.5mm_Pitch0.65mm, symbol STM8S003F3P
- removed P1: CONN_01X06, Pin_Headers:Pin_Header_Straight_1x06, symbol CONN_01X06
- removed P2: USB_OTG, MyOwn:USB_Micro-B_MK5P, symbol USB_OTG
- removed P3, P4: CONN_01X09, Pin_Headers:Pin_Header_Straight_1x09, symbol CONN_01X09
- removed P5: CONN_01X02, Pin_Headers:Pin_Header_Straight_1x02, symbol CONN_01X02
- removed U1: AS1117-5.0, TO_SOT_Packages_SMD:SOT-223, symbol AP1117D33
- removed Y1: 16MHz, Crystals:Crystal_HC49-U_Vertical, symbol Crystal
- added D3: 5.6V, MyOwn:SOD-80, symbol D_Zener
- added J1: CONN_01X04, SparkFun-Connectors:1X04_LOCK, symbol CONN_01X04
- added J2: CONN_02X04, SparkFun-Connectors:2X4, symbol CONN_02X04
- added J3, J4: CONN_01X10, SparkFun-Connectors:1X10_LOCK_NS, symbol CONN_01X10
- added JP2: 12V-30V input, SparkFun-Jumpers:SMT-JUMPER_2_NO_NO-SILK, symbol Jumper_NC_Small
- added Q1: BC817-40, TO_SOT_Packages_SMD:SOT-23, symbol BC817-40
- added R4: 1K, Resistors_SMD:R_0603, symbol R
- added U1: XC6206, TO_SOT_Packages_SMD:SOT-23, symbol APE8865N-33-HF-3
- added U2: STM8S003F3U, MyOwn:UQFN-16_3x3mm_Pitch0.5mm, symbol STM8S003F3U
- C1: footprint Capacitors_SMD:C_0603_HandSoldering -> Capacitors_SMD:C_0603
- C2: renamed from C6; value 10uF -> 1uF; footprint Capacitors_SMD:C_0805_HandSoldering -> Capacitors_SMD:C_0603
- C3: renamed from C2; footprint Capacitors_SMD:C_0603_HandSoldering -> Capacitors_SMD:C_0805
- C4: renamed from C7; value 10uF -> 1uF; footprint Capacitors_SMD:C_0805_HandSoldering -> Capacitors_SMD:C_0603
- C5: renamed from C3; footprint Capacitors_SMD:C_0603_HandSoldering -> Capacitors_SMD:C_0603
- D1, D2: footprint LEDs:LED-0603 -> LEDs:LED_0603
- R1, R2, R3: footprint Resistors_SMD:R_0603_HandSoldering -> Resistors_SMD:R_0603
- SW1: footprint Buttons_Switches_SMD:SW_SPST_EVQPE1 -> Buttons_Switches_SMD:SW_SPST_B3U-1000P
Connections:
- net GND: now also D3.2 (A), J1.3 (P3), J2.1 (P1), J4.1 (P1), U1.1 (GND), U2.4 (VSS)
- net NRST: now also J1.1 (P1), J4.5 (P5), U2.1 (NRST)
- net PA1/OSC_IN: now also J4.4 (P4), U2.2 (OSCIN/PA1)
- net PA2/OSC_OUT: now also J4.3 (P3), U2.3 (OSCOUT/PA2)
- net PA3: now also J2.8 (P8), J3.2 (P2), U2.7 ([SPI_NSS]TIM2_CH3/PA3)
- net PB4: now also J2.3 (P3), J3.4 (P4), U2.9 ([ADC_ETR]I2C_SCL/PB4)
- net PB5: now also J2.4 (P4), J3.3 (P3), U2.8 ([TIM1_BKIN]I2C_SDA/PB5)
- net PC3: now also J3.5 (P5), U2.10 ([TIM1_CH1N]TIM1_CH3/PC3)
- net PC4: now also R2.2, J3.6 (P6), U2.11 ([TIM1_CH2N]AIN2/TIM1_CH4/PC4)
- net PC5: now also J2.5 (P5), J3.7 (P7), U2.12 ([TIM2_CH1]SPI_SCK/PC5)
- net PC6: now also J2.6 (P6), J3.8 (P8), U2.13 ([TIM1_CH1]SPI_MOSI/PC6)
- net PC7: now also J2.7 (P7), J3.9 (P9), U2.14 ([TIM1_CH2]SPI_MISO/PC7)
- net PD1/SWIM: now also J1.2 (P2), J3.10 (P10), U2.15 (PD1/SWIM)
- net PD2: now also J4.10 (P10), U2.16 (PD2/AIN3[TIM2_CH3])
- net PD3: now also J4.9 (P9), U2.17 (PD3/AIN4/TIM2_CH2)
- net PD4: now also J4.8 (P8), U2.18 (PD4/TIM2_CH1/BEEP/UART1_CK); no longer R2.2
- net PD5/TX: now also J4.7 (P7), U2.19 (PD5/AIN5/UART1_TX)
- net PD6/RX: now also J4.6 (P6), U2.20 (PD6/AIN6/UART1_RX)
- net VCC: now also J3.1 (P1), JP2.1, Q1.3 (C), R4.1; no longer C4.1, C5.2, D1.2 (A), D2.2 (A), R1.1
- net at C3.1: now also U2.5 (Vcap)
- net +12V: no longer names the net of C2.1
- net +12V: now also JP2.2, Q1.2 (E), U1.3 (VIN)
- new net: D3.1 (K), Q1.1 (B), R4.2
- new net +3V3: C4.1, C5.2, D1.2 (A), D2.2 (A), J1.4 (P4), J2.2 (P2), J4.2 (P2), R1.1, U1.2 (VOUT), U2.6 (VDD)
- no-connect marks 3 -> 0
Other:
- moved on the sheet: C2, C4
